File: hw/motherboard/main/main.sch (KiCad schematic (older format))
At the start: 20 parts, among them J1 ST-LINK/V2-1, SW1 SW_Push, U1 STM32F373VCTx, Y1 HSE

Commit message: Add RGB leds to schematic
Connections:
- net rgb/DIN: now reaches U1.23 (PA0)
Other:
- note added: "TODO:\n* 5V regulator for leds\n* data output connector for leds\n* power input connector\n* programmer connector\n"
- note removed: "TODO:\n* 5V regulator for leds\n* leds\n* power input connector\n* programmer connector\n"
Changed lines of the file:
@@
 $Descr A4 11693 8268
 encoding utf-8
-Sheet 1 1
+Sheet 1 2
 Title "KAPINE Motherboard"
 Date ""
@@
 $EndComp
 Text Notes 9050 5750 0    50   ~ 0
-TODO:\n* 5V regulator for leds\n* leds\n* power input connector\n* programmer connector\n
+TODO:\n* 5V regulator for leds\n* data output connector for leds\n* power input connector\n* programmer connector\n
 $Comp
 L power:VDDA #PWR03
@@
 Wire Wire Line
 	4350 1450 4300 1450
+$Sheet
+S 8000 1350 550  200
+U 5E444A98
+F0 "rgb" 50
+F1 "rgb.sch" 50
+F2 "DIN" I L 8000 1450 50
+$EndSheet
+Wire Wire Line
+	7450 1450 8000 1450
 $EndSCHEMATC
