File: hw/motherboard/main/main.sch (KiCad schematic (older format))
At the start: 18 parts, among them J1 ST-LINK/V2-1, J2 Conn_ARM_JTAG_SWD_10, SW1 SW_Push, U1 STM32F303RETx, Y1 HSE

Commit message: Add cubemx project for pin configuration.
Parts:
- removed J1: ST-LINK/V2-1, Connector_Molex:Molex_PicoBlade_53261-0671_1x06-1MP_P1.25mm_Horizontal, symbol Connector_Generic_MountingPin:Conn_01x06_MountingPin
- added C12: 4.7u, Capacitor_SMD:C_0603_1608Metric, symbol Device:C_Small
- added C13, C8: 100n, Capacitor_SMD:C_0603_1608Metric, symbol Device:C_Small
- added D33: LED_5V, LED_SMD:LED_0805_2012Metric, symbol Device:LED
- added D34: LED_3V3, LED_SMD:LED_0805_2012Metric, symbol Device:LED
- added D35: LED_TX, symbol Device:LED
- added D36: LED_RX, symbol Device:LED
- added D37: DEBUG_1, LED_SMD:LED_0805_2012Metric, symbol Device:LED
- added D38: DEBUG_2, LED_SMD:LED_0805_2012Metric, symbol Device:LED
- added J1: SWD holes, Connector_PinHeader_2.54mm:PinHeader_1x06_P2.54mm_Vertical, symbol Connector:Conn_01x06_Female
- added J3: USB_B_Mini, symbol Connector:USB_B_Mini
- added J?: STACK_GND, symbol Connector_Generic:Conn_02x02_Counter_Clockwise
- added R10, R11: 1K, Resistor_SMD:R_0805_2012Metric, symbol Device:R
- added R6, R7: TBD, Resistor_SMD:R_0805_2012Metric, symbol Device:R
- added R8, R9: 1k, symbol Device:R
- added U2: FT232RL-REEL, digikey-footprints:SSOP-28_W5.30mm, symbol dk_Interface-Controllers:FT232RL-REEL
- J2: footprint Connector_PinHeader_1.27mm:PinHeader_2x05_P1.27mm_Vertical_SMD -> digikey-footprints:PinHeader_2x5_P1.27mm_Drill.7mm
Connections:
- net labels added: +5V, DEBUG_1, DEBUG_2, JTAG_TCK, JTAG_TDI, JTAG_TDO, JTAG_TMS, RESET#, USART1_RX, USART1_TX, m0, m1, m10, m11, m12, m13, m14, m15, m2, m3, m4, m5, m6, m7, m8, m9
- net labels removed: JTAG_TRST, NRST, boot_sel
- wire segments 79 -> 129
- no-connect marks 2 -> 15
Other:
- note added: "DEBUG LEDs"
- note added: "Electromagnet control signals: m[0..15]\nPhoto gate sensor inputs: s[0..15]"
- note added: "JTAG Programmer"
- note added: "Power Indicators"
- note added: "SWD pins for ST-LINK/V2-1"
- note added: "TODO (Power):\n- Regulators\n * 3V3 digital\n * 3V3 analog\n * 5V logic\n * 5V leds\n- Power routing (usb power to mcu with a jumper)"
- note added: "TODO (Stack):\n- stack connectors\n- em control signals\n- sensor input signals"
- note added: "TODO:\n- Configure as self powered USB device\n (i.e. don't use the usb connector to power on any components)"
- note added: "TODO:\n- Figure out power distribution\n- data output connector for leds\n- power input connector\n"
- note added: "UART-USB Bridge"
- note removed: "Boot select jumper"
- note removed: "Programmer"
- note removed: "TODO JTAG:\n- add jtag labels to programmer connector\n- add jtag labels to mcu\n- verify nrst signal"
- note removed: "TODO: Select crystal"
- note removed: "TODO:\n- 3.3V regulator for MCU \n- 5V regulator for leds\n- data output connector for leds\n- power input connector\n- programmer connector\n"
- moved on the sheet: C1, C10, C11, C2, C3, C4, C5, C6, C7, C9, J2, JP1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

Commit message: WIP Start motherboard PCB layout.
Parts:
- removed J3: USB_B_Mini, symbol Connector:USB_B_Mini
- added J3: 690-005-299-043, digikey-footprints:USB_Mini_B_Female_690-005-299-043, symbol dk_USB-DVI-HDMI-Connectors:690-005-299-043
- D35, D36: footprint (none) -> LED_SMD:LED_0805_2012Metric
- J4: renamed from J?; footprint (none) -> Connector_PinSocket_2.54mm:PinSocket_2x02_P2.54mm_Vertical
- R8, R9: footprint (none) -> Resistor_SMD:R_0805_2012Metric
Connections:
- net labels added: USB_DM, USB_DP, VBUS
- wire segments 129 -> 132
Other:
- note added: "TODO (Layout):\n* Add mounting holes"
- note added: "TODO: usb power connections"
- moved on the sheet: D35, D36, R8, R9
Changed lines of the file:
@@
 	0    -1   -1   0
 $EndComp
-$Comp
-L Connector:USB_B_Mini J3
-U 1 1 5F4812D9
-P 1100 5850
-F 0 "J3" H 1100 6350 50  0000 C CNN
-F 1 "USB_B_Mini" H 1100 6250 50  0000 C CNN
-F 2 "" H 1250 5800 50  0001 C CNN
-F 3 "~" H 1250 5800 50  0001 C CNN
-	1    1100 5850
-	1    0    0    -1
-$EndComp
-Wire Wire Line
-	1100 6250 1000 6250
-$Comp
-L power:GND #PWR0103
-U 1 1 5F48B279
-P 1000 6250
-F 0 "#PWR0103" H 1000 6000 50  0001 C CNN
-F 1 "GND" H 1005 6077 50  0000 C CNN
-F 2 "" H 1000 6250 50  0001 C CNN
-F 3 "" H 1000 6250 50  0001 C CNN
-	1    1000 6250
-	1    0    0    -1
-$EndComp
-Connection ~ 1000 6250
-NoConn ~ 1400 6050
-Wire Wire Line
-	1400 5850 2650 5850
-Wire Wire Line
-	2650 5950 1400 5950
 Wire Wire Line
 	2600 6250 2650 6250
@@
 L power:+5V #PWR0104
 U 1 1 5F51AB08
-P 1550 6400
-F 0 "#PWR0104" H 1550 6250 50  0001 C CNN
-F 1 "+5V" H 1565 6573 50  0000 C CNN
-F 2 "" H 1550 6400 50  0001 C CNN
-F 3 "" H 1550 6400 50  0001 C CNN
-	1    1550 6400
+P 1700 6400
+F 0 "#PWR0104" H 1700 6250 50  0001 C CNN
+F 1 "+5V" H 1715 6573 50  0000 C CNN
+F 2 "" H 1700 6400 50  0001 C CNN
+F 3 "" H 1700 6400 50  0001 C CNN
+	1    1700 6400
 	1    0    0    -1
 $EndComp
@@
 L Device:LED D35
 U 1 1 5F51C9F7
-P 1550 6550
-F 0 "D35" V 1650 6500 50  0000 R CNN
-F 1 "LED_TX" H 1650 6650 50  0000 R CNN
-F 2 "" H 1550 6550 50  0001 C CNN
-F 3 "~" H 1550 6550 50  0001 C CNN
-	1    1550 6550
+P 1700 6550
+F 0 "D35" V 1800 6500 50  0000 R CNN
+F 1 "LED_TX" H 1800 6650 50  0000 R CNN
+F 2 "LED_SMD:LED_0805_2012Metric" H 1700 6550 50  0001 C CNN
+F 3 "~" H 1700 6550 50  0001 C CNN
+	1    1700 6550
 	0    -1   -1   0
 $EndComp
@@
 L Device:R R8
 U 1 1 5F51DAC6
-P 1550 6850
-F 0 "R8" H 1600 6850 50  0000 L CNN
-F 1 "1k" V 1550 6800 50  0000 L CNN
-F 2 "" V 1480 6850 50  0001 C CNN
-F 3 "~" H 1550 6850 50  0001 C CNN
-	1    1550 6850
-	1    0    0    -1
-$EndComp
-Wire Wire Line
-	1550 7000 1550 7150
-Wire Wire Line
-	1550 7150 2650 7150
+P 1700 6850
+F 0 "R8" H 1750 6850 50  0000 L CNN
+F 1 "1k" V 1700 6800 50  0000 L CNN
+F 2 "Resistor_SMD:R_0805_2012Metric" V 1630 6850 50  0001 C CNN
+F 3 "~" H 1700 6850 50  0001 C CNN
+	1    1700 6850
+	1    0    0    -1
+$EndComp
+Wire Wire Line
+	1700 7000 1700 7150
+Wire Wire Line
+	1700 7150 2650 7150
 $Comp
 L power:+5V #PWR0105
 U 1 1 5F52E2B1
-P 1900 6400
-F 0 "#PWR0105" H 1900 6250 50  0001 C CNN
-F 1 "+5V" H 1915 6573 50  0000 C CNN
-F 2 "" H 1900 6400 50  0001 C CNN
-F 3 "" H 1900 6400 50  0001 C CNN
-	1    1900 6400
+P 2050 6400
+F 0 "#PWR0105" H 2050 6250 50  0001 C CNN
+F 1 "+5V" H 2065 6573 50  0000 C CNN
+F 2 "" H 2050 6400 50  0001 C CNN
+F 3 "" H 2050 6400 50  0001 C CNN
+	1    2050 6400
 	1    0    0    -1
 $EndComp
@@
 L Device:LED D36
 U 1 1 5F52E2B7
-P 1900 6550
-F 0 "D36" V 2000 6500 50  0000 R CNN
-F 1 "LED_RX" H 2000 6650 50  0000 R CNN
-F 2 "" H 1900 6550 50  0001 C CNN
-F 3 "~" H 1900 6550 50  0001 C CNN
-	1    1900 6550
+P 2050 6550
+F 0 "D36" V 2150 6500 50  0000 R CNN
+F 1 "LED_RX" H 2150 6650 50  0000 R CNN
+F 2 "LED_SMD:LED_0805_2012Metric" H 2050 6550 50  0001 C CNN
+F 3 "~" H 2050 6550 50  0001 C CNN
+	1    2050 6550
 	0    -1   -1   0
 $EndComp
@@
 L Device:R R9
 U 1 1 5F52E2BD
-P 1900 6850
-F 0 "R9" H 1950 6850 50  0000 L CNN
-F 1 "1k" V 1900 6800 50  0000 L CNN
-F 2 "" V 1830 6850 50  0001 C CNN
-F 3 "~" H 1900 6850 50  0001 C CNN
-	1    1900 6850
-	1    0    0    -1
-$EndComp
-Wire Wire Line
-	1900 7000 1900 7050
-Wire Wire Line
-	1900 7050 2650 7050
+P 2050 6850
+F 0 "R9" H 2100 6850 50  0000 L CNN
+F 1 "1k" V 2050 6800 50  0000 L CNN
+F 2 "Resistor_SMD:R_0805_2012Metric" V 1980 6850 50  0001 C CNN
+F 3 "~" H 2050 6850 50  0001 C CNN
+	1    2050 6850
+	1    0    0    -1
+$EndComp
+Wire Wire Line
+	2050 7000 2050 7050
+Wire Wire Line
+	2050 7050 2650 7050
 NoConn ~ 2650 6350
 Text Notes 550  7700 0    50   ~ 0
@@
 m15
 $Comp
-L power:GND #PWR?
+L power:GND #PWR095
 U 1 1 5F529F84
 P 10700 5550
-F 0 "#PWR?" H 10700 5300 50  0001 C CNN
+F 0 "#PWR095" H 10700 5300 50  0001 C CNN
 F 1 "GND" H 10705 5377 50  0000 C CNN
 F 2 "" H 10700 5550 50  0001 C CNN
@@
 	10700 5550 10700 5500
 $Comp
-L Connector_Generic:Conn_02x02_Counter_Clockwise J?
+L Connector_Generic:Conn_02x02_Counter_Clockwise J4
 U 1 1 5F5307C2
 P 10650 5300
-F 0 "J?" H 10700 5517 50  0000 C CNN
+F 0 "J4" H 10700 5517 50  0000 C CNN
 F 1 "STACK_GND" H 10700 5426 50  0000 C CNN
-F 2 "" H 10650 5300 50  0001 C CNN
+F 2 "Connector_PinSocket_2.54mm:PinSocket_2x02_P2.54mm_Vertical" H 10650 5300 50  0001 C CNN
 F 3 "~" H 10650 5300 50  0001 C CNN
 	1    10650 5300
@@
 Text Notes 8750 5600 0    50   ~ 0
 TODO (Stack):\n- stack connectors\n- em control signals\n- sensor input signals
+$Comp
+L power:PWR_FLAG #FLG02
+U 1 1 5F542403
+P 8850 650
+F 0 "#FLG02" H 8850 725 50  0001 C CNN
+F 1 "PWR_FLAG" V 8850 778 50  0000 L CNN
+F 2 "" H 8850 650 50  0001 C CNN
+F 3 "~" H 8850 650 50  0001 C CNN
+	1    8850 650
+	0    1    1    0
+$EndComp
+$Comp
+L power:VDD #PWR096
+U 1 1 5F561D78
+P 8850 650
+F 0 "#PWR096" H 8850 500 50  0001 C CNN
+F 1 "VDD" V 8850 850 50  0000 C CNN
+F 2 "" H 8850 650 50  0001 C CNN
+F 3 "" H 8850 650 50  0001 C CNN
+	1    8850 650
+	0    -1   -1   0
+$EndComp
+$Comp
+L power:VDDA #PWR0111
+U 1 1 5F57B398
+P 8850 750
+F 0 "#PWR0111" H 8850 600 50  0001 C CNN
+F 1 "VDDA" V 8850 1000 50  0000 C CNN
+F 2 "" H 8850 750 50  0001 C CNN
+F 3 "" H 8850 750 50  0001 C CNN
+	1    8850 750
+	0    -1   -1   0
+$EndComp
+$Comp
+L power:PWR_FLAG #FLG0101
+U 1 1 5F57BC34
+P 8850 750
+F 0 "#FLG0101" H 8850 825 50  0001 C CNN
+F 1 "PWR_FLAG" V 8850 878 50  0000 L CNN
+F 2 "" H 8850 750 50  0001 C CNN
+F 3 "~" H 8850 750 50  0001 C CNN
+	1    8850 750
+	0    1    1    0
+$EndComp
+$Comp
+L power:GND #PWR097
+U 1 1 5F59A129
+P 800 6450
+F 0 "#PWR097" H 800 6200 50  0001 C CNN
+F 1 "GND" H 805 6277 50  0000 C CNN
+F 2 "" H 800 6450 50  0001 C CNN
+F 3 "" H 800 6450 50  0001 C CNN
+	1    800  6450
+	1    0    0    -1
+$EndComp
+$Comp
+L dk_USB-DVI-HDMI-Connectors:690-005-299-043 J3
+U 1 1 5F594174
+P 400 6650
+F 0 "J3" H 1025 8002 60  0000 C CNN
+F 1 "690-005-299-043" H 1025 7896 60  0000 C CNN
+F 2 "digikey-footprints:USB_Mini_B_Female_690-005-299-043" H 600 6850 60  0001 L CNN
+F 3 "http://files.edac.net/690-005-299-043.pdf" H 600 6950 60  0001 L CNN
+F 4 "151-1206-1-ND" H 600 7050 60  0001 L CNN "Digi-Key_PN"
+F 5 "690-005-299-043" H 600 7150 60  0001 L CNN "MPN"
+F 6 "Connectors, Interconnects" H 600 7250 60  0001 L CNN "Category"
+F 7 "USB, DVI, HDMI Connectors" H 600 7350 60  0001 L CNN "Family"
+F 8 "http://files.edac.net/690-005-299-043.pdf" H 600 7450 60  0001 L CNN "DK_Datasheet_Link"
+F 9 "/product-detail/en/edac-inc/690-005-299-043/151-1206-1-ND/4312192" H 600 7550 60  0001 L CNN "DK_Detail_Page"
+F 10 "CONN RCPT USB2.0 MINI B SMD R/A" H 600 7650 60  0001 L CNN "Description"
+F 11 "EDAC Inc." H 600 7750 60  0001 L CNN "Manufacturer"
+F 12 "Active" H 600 7850 60  0001 L CNN "Status"
+	1    400  6650
+	1    0    0    -1
+$EndComp
+Text Label 1350 5950 0    50   ~ 0
+USB_DP
+Wire Wire Line
+	1350 5950 1300 5950
+Text Label 1350 5850 0    50   ~ 0
+USB_DM
+Wire Wire Line
+	1350 5850 1300 5850
+$Comp
+L power:GND #PWR099
+U 1 1 5F5B9D07
+P 1350 6150
+F 0 "#PWR099" H 1350 5900 50  0001 C CNN
+F 1 "GND" H 1355 5977 50  0000 C CNN
+F 2 "" H 1350 6150 50  0001 C CNN
+F 3 "" H 1350 6150 50  0001 C CNN
+	1    1350 6150
+	1    0    0    -1
+$EndComp
+Wire Wire Line
+	1350 6150 1300 6150
+NoConn ~ 1300 6050
+Text Label 2600 5850 2    50   ~ 0
+USB_DP
+Wire Wire Line
+	2600 5850 2650 5850
+Text Label 2600 5950 2    50   ~ 0
+USB_DM
+Wire Wire Line
+	2600 5950 2650 5950
+Wire Wire Line
+	1300 5750 1350 5750
+$Comp
+L power:VBUS #PWR098
+U 1 1 5F5FFEA6
+P 1350 5750
+F 0 "#PWR098" H 1350 5600 50  0001 C CNN
+F 1 "VBUS" H 1365 5923 50  0000 C CNN
+F 2 "" H 1350 5750 50  0001 C CNN
+F 3 "" H 1350 5750 50  0001 C CNN
+	1    1350 5750
+	1    0    0    -1
+$EndComp
+Text Notes 1250 5550 0    50   ~ 0
+TODO: usb power connections
+Text Notes 8500 4700 0    50   ~ 0
+TODO (Layout):\n* Add mounting holes
 $EndSCHEMATC

Commit message: WIP Add electromagnet and sensor schematic connections to MCU pins
Parts:
- removed C12: 4.7u, Capacitor_SMD:C_0603_1608Metric, symbol Device:C_Small
- removed C13, C8: 100n, Capacitor_SMD:C_0603_1608Metric, symbol Device:C_Small
- removed D33: LED_5V, LED_SMD:LED_0805_2012Metric, symbol Device:LED
- removed D34: LED_3V3, LED_SMD:LED_0805_2012Metric, symbol Device:LED
- removed D35: LED_TX, LED_SMD:LED_0805_2012Metric, symbol Device:LED
- removed D36: LED_RX, LED_SMD:LED_0805_2012Metric, symbol Device:LED
- removed J3: 690-005-299-043, digikey-footprints:USB_Mini_B_Female_690-005-299-043, symbol dk_USB-DVI-HDMI-Connectors:690-005-299-043
- removed R6, R7: TBD, Resistor_SMD:R_0805_2012Metric, symbol Device:R
- removed R8, R9: 1k, Resistor_SMD:R_0805_2012Metric, symbol Device:R
- removed U2: FT232RL-REEL, digikey-footprints:SSOP-28_W5.30mm, symbol dk_Interface-Controllers:FT232RL-REEL
- added H1, H2, H3, H4: MountingHole, MountingHole:MountingHole_4.3mm_M4, symbol Mechanical:MountingHole
Connections:
- net labels added: em0, em1, em10, em11, em12, em13, em14, em15, em2, em3, em4, em5, em6, em7, em8, em9, s0, s1, s10, s11, s12, s13, s14, s15, s2, s3, s4, s5, s6, s7, s8, s9
- net labels removed: +5V, USB_DM, USB_DP, VBUS, m0, m1, m10, m11, m12, m13, m14, m15, m2, m3, m4, m5, m6, m7, m8, m9
- wire segments 132 -> 129
- no-connect marks 15 -> 8
Other:
- note added: "Electromagnet control signals: em[0..15]\nPhoto gate sensor inputs: s[0..15]"
- note removed: "Electromagnet control signals: m[0..15]\nPhoto gate sensor inputs: s[0..15]"
- note removed: "Power Indicators"
- note removed: "TODO (Layout):\n* Add mounting holes"
- note removed: "TODO (Power):\n- Regulators\n * 3V3 digital\n * 3V3 analog\n * 5V logic\n * 5V leds\n- Power routing (usb power to mcu with a jumper)"
- note removed: "TODO: usb power connections"
- note removed: "TODO:\n- Configure as self powered USB device\n (i.e. don't use the usb connector to power on any components)"
- note removed: "TODO:\n- Figure out power distribution\n- data output connector for leds\n- power input connector\n"
- note removed: "UART-USB Bridge"
- moved on the sheet: C1, C10, C11, C2, C3, C4, C5, C6, C7, C9, JP1, R1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
