File: hw/motherboard/main/uart.sch (KiCad schematic (older format))
At the start: 17 parts, among them J3 690-005-299-043, J7 UART pins, J8 CBUS[2..4], U2 USBLC6-2SC6, U5 FT232RL-REEL

Commit message: Minor motherboard layout changes. Bump revision number to 1.1.
Other:
- note removed: "TODO: Configure as bus powered\n- Protection circuitry\n- Configuration jumper for MCU power from USB"
Changed lines of the file:
@@
 encoding utf-8
 Sheet 4 4
-Title "KAPINE Motherboard UART"
-Date ""
-Rev ""
+Title "KAPINE Motherboard"
+Date "2020-09-02"
+Rev "1.1"
 Comp "Verneri Hirvonen"
 Comment1 ""
@@
 	1    0    0    -1
 $EndComp
-Text Notes 9000 850  0    50   ~ 0
-TODO: Configure as bus powered\n- Protection circuitry\n- Configuration jumper for MCU power from USB
 Wire Wire Line
 	7050 3500 7800 3500

Commit message: Add missing component values.
Parts:
- C12: footprint Capacitor_SMD:C_0603_1608Metric -> Capacitor_SMD:C_0805_2012Metric
Changed lines of the file:
@@
 F 0 "C12" H 4492 4896 50  0000 L CNN
 F 1 "4.7u" H 4492 4805 50  0000 L CNN
-F 2 "Capacitor_SMD:C_0603_1608Metric" H 4400 4850 50  0001 C CNN
+F 2 "Capacitor_SMD:C_0805_2012Metric" H 4400 4850 50  0001 C CNN
 F 3 "~" H 4400 4850 50  0001 C CNN
 	1    4400 4850

Commit message: wip: fix motherboard v1.1 bugs
Parts:
- U2: symbol Power_Protection:USBLC6-2SC6 -> main-rescue:USBLC6-2SC6-Power_Protection
Changed lines of the file:
@@
 $EndComp
 $Comp
-L Power_Protection:USBLC6-2SC6 U?
+L main-rescue:USBLC6-2SC6-Power_Protection U?
 U 1 1 5F5A6BBF
 P 4500 3100
