File: hw/motherboard/main/main.kicad_pcb (KiCad board)
At the start: 4 copper layers, 100 x 100 mm, 132 parts, among them J1 SWD holes, J10 stack[0..3], J11 stack[0..3], J12 stack[0..3], J13 GPIO, J2 Conn_ARM_JTAG_SWD_10, J3 690-005-299-043, J4 STACK_GND, J5 RGB stack, J6 STACK_5V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

Commit message: Update KiCad files to KiCad 8
Routing:
- added copper zone on In2.Cu, net GND
- added copper zone on In1.Cu, net VDD
- removed copper zone on GND, net GND
- removed copper zone on VDD, net VDD
Other:
- net class Default removed
