File: hw/relelauta/v2/relelauta/relelauta.kicad_pcb (KiCad board)
At the start: 2 copper layers, 100 x 100 mm, 150 parts, among them J1 stack[0..3], J10 PSU_Conn, J11 Conn_sensor, J12 Conn_sensor, J13 Conn_sensor, J14 Conn_sensor, J15 Conn_sensor, J16 Conn_sensor, J17 Conn_sensor, J18 Conn_sensor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

Commit message: Update KiCad files to KiCad 8
Other:
- net class Default removed
