File: hw/sensorilauta/sensorilauta.kicad_pcb (KiCad board)
At the start: 2 copper layers, 29.2 x 29.5 mm, 16 parts, among them J1 motherboard connector, Q1 Q_Photo_NPN, U1 MCP6001U

Commit message: Update sensorilauta files to KiCad 8
Other:
- net class Default removed
